File: LiIon_Charger.kicad_pcb (KiCad board)
At the start: 2 copper layers, 19 x 20 mm, 35 parts, among them U1 MP26123, j1 Conn_01x01, j2 Conn_01x01, j3 Conn_01x01, j4 Conn_01x01, j5 Conn_01x01, j6 Conn_01x01

Commit message: V1 Ordered
Parts:
- moved D3 0.09 mm to (141.4, 83.5)
Routing:
- net /Charger: track 1.49 -> 6.04 mm, vias 0 -> 2
- net Net-(U1-Pad6): track 12.5 -> 15.3 mm, vias 0 -> 1
- net /NTC: track 8.95 -> 11.6 mm, vias 0 -> 1
- net /~{CHGOK}: track 13.3 -> 15.9 mm, vias 0 -> 1
- net /Battery: track 9.52 -> 12.0 mm, vias 0 -> 1
- net /~{ACOK}: track 13.2 -> 14.6 mm, vias 2 -> 3
- net GND: vias 19 -> 22
Other:
- board text added: "CHARGE"
- board text added: "POWER"
- board text added: "~{EN}"
- board text removed: "LED1"
- board text removed: "LED2"
- board text removed: "__ EN"
